File: kicad/4164-41256-tester.kicad_pcb (KiCad board)
At the start: 2 copper layers, 76.2 x 43.7 mm, 34 parts, among them J1 Jack-DC, J2 Conn_01x02, J3 ZIF-16, J4 Display, J5 Serial, J6 ICSP, SW1 SW_Push, SW2 SW_Push, SW3 SW_Push, U1 AMS1117-5.0

Commit message: add ibom
Parts:
- A1: value Arduino_Pro_Mini -> Arduino Pro Mini
- C1, C3, C4: value C -> 100 nF
- C2: value C_Polarized -> 1000 uF
- J1: value Jack-DC -> Jack DC
- J2: value Conn_01x02 -> PCB Terminal Block
- R1, R10, R11, R12, R13, R2, R3, R4, R5, R6, R7, R8, R9: value R -> 47
- R14, R15: value R -> 10K
- SW1, SW2, SW3: value SW_Push -> SW Push
