File: kicad/4164-41256-tester.kicad_sch (KiCad schematic)
At the start: 30 parts, among them J1 Jack-DC, J2 Conn_01x02, J3 ZIF-16, J4 Display, J5 Serial, J6 ICSP, SW1 SW_Push, SW2 SW_Push, SW3 SW_Push, U1 AMS1117-5.0

Commit message: add ibom
Parts:
- A1: value Arduino_Pro_Mini -> Arduino Pro Mini; Link (none) -> https://aliexpress.ru/item/32849721150.html?af=1954_7685&cn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
- C1, C3, C4: value C -> 100 nF; Link (none) -> https://aliexpress.ru/item/33007425729.html?sku_id=67085457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; Note (none) -> smd 0805
- C2: value C_Polarized -> 1000 uF; Link (none) -> https://aliexpress.ru/item/4001227639043.html?sku_id=100000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
- J1: value Jack-DC -> Jack DC; Link (none) -> https://aliexpress.ru/item/32361314769.html?spm=a2g2w.order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
- J2: value Conn_01x02 -> PCB Terminal Block; Link (none) -> https://aliexpress.ru/item/4000290521933.html?sku_id=100000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
- J3: Link (none) -> https://aliexpress.ru/item/1005002108879940.html?spm=a2g2w.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
- J4: Link (none) -> https://aliexpress.ru/item/32672327708.html?spm=a2g2w.order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; Note (none) -> 0,91 OLED 128X32
- J5: Link (none) -> https://aliexpress.ru/item/32849370527.html?spm=a2g2w.order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; Note (none) -> 1x4
- J6: Link (none) -> https://aliexpress.ru/item/32848766148.html?spm=a2g2w.order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; Note (none) -> 2x3
- R1, R10, R11, R12, R13, R2, R3, R4, R5, R6, R7, R8, R9: value R -> 47; Link (none) -> https://aliexpress.ru/item/1005001625934589.html?spm=a2g2w.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; Note (none) -> smd 0805
- R14, R15: value R -> 10K; Link (none) -> https://aliexpress.ru/item/1005001625934589.html?spm=a2g2w.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; Note (none) -> smd 0805
- SW1, SW2, SW3: value SW_Push -> SW Push; Link (none) -> https://aliexpress.ru/item/32912263133.html?sku_id=65911938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; Note (none) -> 6 mm
- U1: Link (none) -> https://aliexpress.ru/item/32868348278.html?af=1954_7685&cn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; Note (none) -> sot-223
